Commit message: feat: add Gazebo simulation launch scaffold

File: colcon_ws/src/aim_arm_description/urdf/aim_arm.urdf.xacro (robot description, xacro)
@@ -98,4 +98,7 @@
     <xacro:visual_collision_cylinder radius="${base_radius}" length="${base_height}" material="mat_base"/>
   </link>
+  <gazebo reference="base_link">
+    <material>Gazebo/DarkGrey</material>
+  </gazebo>
   <joint name="shoulder_pan_joint" type="revolute">
     <parent link="base_link"/>
@@ -110,4 +113,7 @@
     <xacro:visual_collision_cylinder radius="0.09" length="${shoulder_height}" material="mat_joint"/>
   </link>
+  <gazebo reference="shoulder_link">
+    <material>Gazebo/White</material>
+  </gazebo>
   <joint name="shoulder_lift_joint" type="revolute">
     <parent link="shoulder_link"/>
@@ -134,4 +140,7 @@
     </collision>
   </link>
+  <gazebo reference="upper_arm_link">
+    <material>Gazebo/Blue</material>
+  </gazebo>
   <joint name="elbow_joint" type="revolute">
     <parent link="upper_arm_link"/>
@@ -158,4 +167,7 @@
     </collision>
   </link>
+  <gazebo reference="forearm_link">
+    <material>Gazebo/Blue</material>
+  </gazebo>
   <joint name="wrist_pitch_joint" type="revolute">
     <parent link="forearm_link"/>
@@ -182,4 +194,7 @@
     </collision>
   </link>
+  <gazebo reference="wrist_pitch_link">
+    <material>Gazebo/White</material>
+  </gazebo>
   <joint name="wrist_roll_joint" type="revolute">
     <parent link="wrist_pitch_link"/>
@@ -206,4 +221,7 @@
     </collision>
   </link>
+  <gazebo reference="wrist_roll_link">
+    <material>Gazebo/White</material>
+  </gazebo>
   <joint name="wrist_yaw_joint" type="revolute">
     <parent link="wrist_roll_link"/>
@@ -230,4 +248,7 @@
     </collision>
   </link>
+  <gazebo reference="tool_link">
+    <material>Gazebo/Orange</material>
+  </gazebo>
   <joint name="tool0_fixed_joint" type="fixed">
     <parent link="tool_link"/>

Commit message: feat: scaffold optional ros2 control integration

File: colcon_ws/src/aim_arm_description/urdf/aim_arm.urdf.xacro (robot description, xacro)
@@ -1,4 +1,6 @@
 <?xml version="1.0"?>
 <robot xmlns:xacro="http://www.ros.org/wiki/xacro" name="aim_arm">
+  <xacro:arg name="enable_ros2_control" default="false"/>
+  <xacro:arg name="ros2_control_config" default="package://aim_arm_description/config/ros2_controllers.yaml"/>
   <xacro:property name="aim_pi" value="3.141592653589793"/>
   <xacro:property name="base_height" value="0.12"/>
@@ -257,3 +259,63 @@
   </joint>
   <link name="tool0"/>
+  <xacro:if value="$(arg enable_ros2_control)">
+    <ros2_control name="AimArmSystem" type="system">
+      <hardware>
+        <plugin>gazebo_ros2_control/GazeboSystem</plugin>
+      </hardware>
+      <joint name="shoulder_pan_joint">
+        <command_interface name="position">
+          <param name="min">-3.14159</param>
+          <param name="max">3.14159</param>
+        </command_interface>
+        <state_interface name="position"/>
+        <state_interface name="velocity"/>
+      </joint>
+      <joint name="shoulder_lift_joint">
+        <command_interface name="position">
+          <param name="min">-2.35619</param>
+          <param name="max">2.35619</param>
+        </command_interface>
+        <state_interface name="position"/>
+        <state_interface name="velocity"/>
+      </joint>
+      <joint name="elbow_joint">
+        <command_interface name="position">
+          <param name="min">-2.61799</param>
+          <param name="max">2.61799</param>
+        </command_interface>
+        <state_interface name="position"/>
+        <state_interface name="velocity"/>
+      </joint>
+      <joint name="wrist_pitch_joint">
+        <command_interface name="position">
+          <param name="min">-3.14159</param>
+          <param name="max">3.14159</param>
+        </command_interface>
+        <state_interface name="position"/>
+        <state_interface name="velocity"/>
+      </joint>
+      <joint name="wrist_roll_joint">
+        <command_interface name="position">
+          <param name="min">-3.14159</param>
+          <param name="max">3.14159</param>
+        </command_interface>
+        <state_interface name="position"/>
+        <state_interface name="velocity"/>
+      </joint>
+      <joint name="wrist_yaw_joint">
+        <command_interface name="position">
+          <param name="min">-3.14159</param>
+          <param name="max">3.14159</param>
+        </command_interface>
+        <state_interface name="position"/>
+        <state_interface name="velocity"/>
+      </joint>
+    </ros2_control>
+    <gazebo>
+      <plugin filename="libgazebo_ros2_control.so" name="gazebo_ros2_control">
+        <parameters>$(arg ros2_control_config)</parameters>
+      </plugin>
+    </gazebo>
+  </xacro:if>
 </robot>

Commit message: feat: use mesh visuals in arm URDF

File: colcon_ws/src/aim_arm_description/urdf/aim_arm.urdf.xacro (robot description, xacro)
@@ -113,5 +113,17 @@
   <link name="shoulder_link">
     <xacro:cylinder_inertia mass="4.0" radius="0.09" length="${shoulder_height}" axis="z"/>
-    <xacro:visual_collision_cylinder radius="0.09" length="${shoulder_height}" material="mat_joint"/>
+    <visual>
+      <origin xyz="0 0 0" rpy="0 ${aim_pi / 2.0} 0"/>
+      <geometry>
+        <mesh filename="package://aim_arm_description/meshes/visual/joint_cap_visual.stl"/>
+      </geometry>
+      <material name="mat_joint"/>
+    </visual>
+    <collision>
+      <origin xyz="0 0 0" rpy="0 0 0"/>
+      <geometry>
+        <cylinder radius="0.09" length="${shoulder_height}"/>
+      </geometry>
+    </collision>
   </link>
   <gazebo reference="shoulder_link">
@@ -129,7 +141,7 @@
     <xacro:box_inertia mass="3.2" x="${upper_arm_length}" y="0.08" z="0.08"/>
     <visual>
-      <origin xyz="${upper_arm_length / 2.0} 0 0" rpy="0 0 0"/>
-      <geometry>
-        <box size="${upper_arm_length} 0.08 0.08"/>
+      <origin xyz="0 0 0" rpy="0 0 0"/>
+      <geometry>
+        <mesh filename="package://aim_arm_description/meshes/visual/upper_arm_visual.stl"/>
       </geometry>
       <material name="mat_link"/>
@@ -156,7 +168,7 @@
     <xacro:box_inertia mass="2.4" x="${forearm_length}" y="0.065" z="0.065"/>
     <visual>
-      <origin xyz="${forearm_length / 2.0} 0 0" rpy="0 0 0"/>
-      <geometry>
-        <box size="${forearm_length} 0.065 0.065"/>
+      <origin xyz="0 0 0" rpy="0 0 0"/>
+      <geometry>
+        <mesh filename="package://aim_arm_description/meshes/visual/forearm_visual.stl"/>
       </geometry>
       <material name="mat_link"/>
@@ -183,7 +195,7 @@
     <xacro:cylinder_inertia mass="0.9" radius="0.055" length="${wrist_length}" axis="x"/>
     <visual>
-      <origin xyz="${wrist_length / 2.0} 0 0" rpy="0 ${aim_pi / 2.0} 0"/>
-      <geometry>
-        <cylinder radius="0.055" length="${wrist_length}"/>
+      <origin xyz="${wrist_length / 2.0} 0 0" rpy="0 0 0"/>
+      <geometry>
+        <mesh filename="package://aim_arm_description/meshes/visual/wrist_visual.stl" scale="0.875 1 1"/>
       </geometry>
       <material name="mat_joint"/>
@@ -210,7 +222,7 @@
     <xacro:cylinder_inertia mass="0.7" radius="0.045" length="0.10" axis="x"/>
     <visual>
-      <origin xyz="0.05 0 0" rpy="0 ${aim_pi / 2.0} 0"/>
-      <geometry>
-        <cylinder radius="0.045" length="0.10"/>
+      <origin xyz="0.05 0 0" rpy="0 0 0"/>
+      <geometry>
+        <mesh filename="package://aim_arm_description/meshes/visual/wrist_visual.stl" scale="0.625 0.9 0.9"/>
       </geometry>
       <material name="mat_joint"/>
@@ -237,7 +249,7 @@
     <xacro:box_inertia mass="0.4" x="${tool_length}" y="0.04" z="0.04"/>
     <visual>
-      <origin xyz="${tool_length / 2.0} 0 0" rpy="0 0 0"/>
-      <geometry>
-        <box size="${tool_length} 0.04 0.04"/>
+      <origin xyz="0 0 0" rpy="0 0 0"/>
+      <geometry>
+        <mesh filename="package://aim_arm_description/meshes/visual/tool_visual.stl" scale="0.625 1 1"/>
       </geometry>
       <material name="mat_tool"/>
